Commit message: Add files via upload

File: urdf/robot.urdf (robot description, URDF)
Before this commit: robot simpleRobot, 5 links, 4 joints
Links:
- link base_link: geometry visual box size=${width} 0.2 0.02
Joints:
- joint base_to_roue_droite: type fixed -> continious
- joint base_to_roue_gauche: type fixed -> continuous
